Commit message: urdf changes includinf tf_prefix fix

File: ur_atc_robot_cell/ur_atc_robot_cell_description/urdf/my_robot_cell_macro.xacro (robot description, xacro)
@@ -3,9 +3,10 @@
   <xacro:include filename="$(find ur_description)/urdf/ur_macro.xacro"/>
   <xacro:include filename="$(find ur_atc_robot_cell_description)/urdf/tool_rack.xacro"/>
-  <xacro:include filename="$(find ur_atc_robot_cell_description)/urdf/gripper_side_TC.xacro" />
+  <xacro:include filename="$(find ur_atc_robot_cell_description)/urdf/gripper_side_tc_scad.xacro" />
   <xacro:macro name="my_robot_cell" params="
     parent
     *origin
     ur_type
+    tf_prefix
     joint_limits_parameters_file
     kinematics_parameters_file
@@ -27,5 +28,6 @@
       <collision>
         <geometry>
-          <mesh filename="package://ur_atc_robot_cell_description/meshes/table.dae"/>
+          <!-- <mesh filename="package://ur_atc_robot_cell_description/meshes/table.dae"/> -->
+          <box size="1.5 1.55 0.84" />
         </geometry>
         <origin rpy="0 0 0" xyz="0.75 0.775 -0.84"/>
@@ -44,5 +46,5 @@
     <xacro:ur_robot
       name="${ur_type}"
-      tf_prefix="${ur_type}_"
+      tf_prefix="${tf_prefix}"
       parent="robot_mount"
       joint_limits_parameters_file="${joint_limits_parameters_file}"
@@ -56,5 +58,5 @@
     <xacro:property name="tool_rack_y_dist" value="0.23" />
     <link name="tool_rack_base"/>
-    <joint name="tool_rack_base" type="fixed">
+    <joint name="tool_rack_base_joint" type="fixed">
       <parent link="table" />
       <child link="tool_rack_base" />

Commit message: changes to fix issues with gazebo sim, working with JTC, scaled JTC and cartesian motion controller

File: ur_atc_robot_cell/ur_atc_robot_cell_description/urdf/my_robot_cell_macro.xacro (robot description, xacro)
@@ -3,5 +3,5 @@
   <xacro:include filename="$(find ur_description)/urdf/ur_macro.xacro"/>
   <xacro:include filename="$(find ur_atc_robot_cell_description)/urdf/tool_rack.xacro"/>
-  <xacro:include filename="$(find ur_atc_robot_cell_description)/urdf/gripper_side_tc_scad.xacro" />
+  <xacro:include filename="$(find ur_atc_robot_cell_description)/urdf/gripper_side_TC.xacro" />
   <xacro:macro name="my_robot_cell" params="
     parent
@@ -31,5 +31,5 @@
           <box size="1.5 1.55 0.84" />
         </geometry>
-        <origin rpy="0 0 0" xyz="0.75 0.775 -0.84"/>
+        <origin rpy="0 0 0" xyz="0.75 0.775 -0.42"/>
       </collision>
     </link>

File: ur_atc_robot_cell/ur_atc_robot_cell_description/urdf/tool_rack.xacro (robot description, xacro)
@@ -28,4 +28,10 @@
                 <material name="blue" />
             </visual>
+            <collision>
+                <origin xyz="0 0 ${C/2}" rpy="0 0 0" />
+                <geometry>
+                    <box size="${D1} ${C} ${C}" />
+                </geometry>
+            </collision>
         </link>
         <link name="ground2_link">
@@ -37,4 +43,10 @@
                 <material name="blue" />
             </visual>
+            <collision>
+                <origin xyz="0 ${W} ${C/2}" rpy="0 0 0" />
+                <geometry>
+                    <box size="${D1} ${C} ${C}" />
+                </geometry>
+            </collision>
         </link>
         <link name="vertical_link">
@@ -46,4 +58,10 @@
                 <material name="green" />
             </visual>
+            <collision>
+                <origin xyz="0 0 ${H/2}" rpy="0 0 0" />
+                <geometry>
+                    <box size="${C} ${C} ${H}" />
+                </geometry>
+            </collision>
         </link>
         <link name="vertical2_link">
@@ -55,4 +73,10 @@
                 <material name="green" />
             </visual>
+            <collision>
+                <origin xyz="0 ${W} ${H/2}" rpy="0 0 0" />
+                <geometry>
+                    <box size="${C} ${C} ${H}" />
+                </geometry>
+            </collision>
         </link>
         <link name="horizontal_link">
@@ -64,4 +88,10 @@
                 <material name="red" />
             </visual>
+            <collision>
+                <origin xyz="0 ${W/2} ${H}" rpy="0 0 0" />
+                <geometry>
+                    <box size="${C} ${W} ${C}" />
+                </geometry>
+            </collision>
         </link>
         <link name="air_link">
@@ -73,4 +103,10 @@
                 <material name="blue" />
             </visual>
+            <collision>
+                <origin xyz="${D2/2} ${W/3} ${H}" rpy="0 0 0" />
+                <geometry>
+                    <box size="${D2} ${C} ${C}" />
+                </geometry>
+            </collision>
         </link>
         <link name="ratelier_link"/>
